Commit message: Update Gazebo simulation config, spawn command, and integrate new robot STLs

File: sim/vector_description/urdf/vector.ros2_control.xacro (robot description, xacro)
@@ -5,13 +5,5 @@
       <plugin>gz_ros2_control/GazeboSimSystem</plugin>
     </hardware>
-    <!-- Torso -->
-    <joint name="slider_z_axis">
-      <command_interface name="effort"/>
-      <state_interface name="position"/>
-      <state_interface name="velocity"/>
-      <state_interface name="effort"/>
-    </joint>
-    <!-- Left Arm -->
-    <joint name="left_shoulder_holder">
+    <joint name="revolute_1">
       <command_interface name="position"/>
       <state_interface name="position">
@@ -20,5 +12,5 @@
       <state_interface name="velocity"/>
     </joint>
-    <joint name="left_shoulder">
+    <joint name="revolute_2">
       <command_interface name="position"/>
       <state_interface name="position">
@@ -27,131 +19,4 @@
       <state_interface name="velocity"/>
     </joint>
-    <joint name="left_bicep">
-      <command_interface name="position"/>
-      <state_interface name="position">
-        <param name="initial_value">0.0</param>
-      </state_interface>
-      <state_interface name="velocity"/>
-    </joint>
-    <joint name="left_forearm">
-      <command_interface name="position"/>
-      <state_interface name="position">
-        <param name="initial_value">0.0</param>
-      </state_interface>
-      <state_interface name="velocity"/>
-    </joint>
-    <!-- Right Arm -->
-    <joint name="right_shoulder_holder">
-      <command_interface name="position"/>
-      <state_interface name="position">
-        <param name="initial_value">0.0</param>
-      </state_interface>
-      <state_interface name="velocity"/>
-    </joint>
-    <joint name="right_shoulder">
-      <command_interface name="position"/>
-      <state_interface name="position">
-        <param name="initial_value">0.0</param>
-      </state_interface>
-      <state_interface name="velocity"/>
-    </joint>
-    <joint name="right_bicep">
-      <command_interface name="position"/>
-      <state_interface name="position">
-        <param name="initial_value">0.0</param>
-      </state_interface>
-      <state_interface name="velocity"/>
-    </joint>
-    <joint name="right_forearn">
-      <command_interface name="position"/>
-      <state_interface name="position">
-        <param name="initial_value">0.0</param>
-      </state_interface>
-      <state_interface name="velocity"/>
-    </joint>
-    <!-- Neck and Head -->
-    <joint name="neck">
-      <command_interface name="position"/>
-      <state_interface name="position">
-        <param name="initial_value">0.0</param>
-      </state_interface>
-      <state_interface name="velocity"/>
-    </joint>
-    <joint name="head">
-      <command_interface name="position"/>
-      <state_interface name="position">
-        <param name="initial_value">0.0</param>
-      </state_interface>
-      <state_interface name="velocity"/>
-    </joint>
-    <!-- Wrists -->
-    <joint name="left_wrist_pitch">
-      <command_interface name="position"/>
-      <state_interface name="position">
-        <param name="initial_value">0.0</param>
-      </state_interface>
-      <state_interface name="velocity"/>
-    </joint>
-    <joint name="left_wrist_yaw">
-      <command_interface name="position"/>
-      <state_interface name="position">
-        <param name="initial_value">0.0</param>
-      </state_interface>
-      <state_interface name="velocity"/>
-    </joint>
-    <joint name="right_wrist_pitch">
-      <command_interface name="position"/>
-      <state_interface name="position">
-        <param name="initial_value">0.0</param>
-      </state_interface>
-      <state_interface name="velocity"/>
-    </joint>
-    <joint name="right_wrist_yaw">
-      <command_interface name="position"/>
-      <state_interface name="position">
-        <param name="initial_value">0.0</param>
-      </state_interface>
-      <state_interface name="velocity"/>
-    </joint>
-    <!-- Hands -->
-    <joint name="left_hand_palm">
-      <command_interface name="position"/>
-      <state_interface name="position">
-        <param name="initial_value">0.0</param>
-      </state_interface>
-      <state_interface name="velocity"/>
-    </joint>
-    <joint name="left_hand_finger">
-      <command_interface name="position"/>
-      <state_interface name="position">
-        <param name="initial_value">0.0</param>
-      </state_interface>
-      <state_interface name="velocity"/>
-    </joint>
-    <joint name="right_hand_palm">
-      <command_interface name="position"/>
-      <state_interface name="position">
-        <param name="initial_value">0.0</param>
-      </state_interface>
-      <state_interface name="velocity"/>
-    </joint>
-    <joint name="right_hand_finger">
-      <command_interface name="position"/>
-      <state_interface name="position">
-        <param name="initial_value">0.0</param>
-      </state_interface>
-      <state_interface name="velocity"/>
-    </joint>
-    <!-- Wheels -->
-    <joint name="right_wheel">
-      <command_interface name="velocity"/>
-      <state_interface name="position"/>
-      <state_interface name="velocity"/>
-    </joint>
-    <joint name="left_wheel">
-      <command_interface name="velocity"/>
-      <state_interface name="position"/>
-      <state_interface name="velocity"/>
-    </joint>
   </ros2_control>
 </robot>

File: sim/vector_description/urdf/vector.urdf (robot description, URDF)
Before this commit: robot vector, 20 links, 19 joints
Links:
- removed link base_link
- removed link camera_1
- removed link head_v1_1
- removed link left_arm_link_1_1
- removed link left_bicep_1
- removed link left_forearm_v2_1
- removed link left_hand_finger_1
- removed link left_hand_palm_1
- removed link left_shoulder_1
- removed link left_wheel_1
- removed link neck_v2_1
- removed link right_arm_link_1_1
- removed link right_bicep_1
- removed link right_forearm_v1_1
- removed link right_hand_finger_1
- removed link right_hand_palm_1
- removed link right_shoulder_1
- removed link right_wheel_1
- removed link slider_1
- removed link torso_1
- added link 9_1_gearbox_from_mas_automation, mass 2.84999; visual mesh filename=package://vector_description/meshes/_9_1_Gearbox_from_MAS_A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 scale=1 1 1
- added link 9_1_gearbox_from_mas_automation_1, mass 2.84999; visual mesh filename=package://vector_description/meshes/_9_1_Gearbox_from_MAS_A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 scale=1 1 1
- added link part_1, mass 0.795632; visual mesh filename=package://vector_description/meshes/Part_1.stl scale=1 1 1
- added link part_1_1, mass 0.795632; visual mesh filename=package://vector_description/meshes/Part_1.stl scale=1 1 1
- added link root; visual mesh filename=package://vector_description/meshes/Back_top_plate.stl scale=1 1 1; visual mesh filename=package://vector_description/meshes/Belt.stl scale=1 1 1
Joints:
- removed joint camera
- removed joint head
- removed joint left_bicep
- removed joint left_forearm
- removed joint left_hand_finger
- removed joint left_hand_palm
- removed joint left_shoulder
- removed joint left_shoulder_holder
- removed joint left_wheel
- removed joint neck
- removed joint right_bicep
- removed joint right_forearn
- removed joint right_hand_finger
- removed joint right_hand_palm
- removed joint right_shoulder
- removed joint right_shoulder_holder
- removed joint right_wheel
- removed joint slider_z_axis
- removed joint torso_with_slider
- added joint hanging_node_to_root_joint: type fixed, parent root, child 9_1_gearbox_from_mas_automation_1, origin xyz=-0.149164 0.134455 -0.0890278 rpy=0 -0 1.5708, axis 0 0 1
- added joint hanging_node_to_root_joint_1: type fixed, parent root, child part_1, origin xyz=0.269068 0.134455 -0.0890278 rpy=0 0 -1.5708, axis 0 0 1
- added joint revolute_1: type revolute, parent 9_1_gearbox_from_mas_automation_1, child part_1_1, origin xyz=0 0.037 0 rpy=3.14159 -2.46519e-32 3.14159, axis 0 -1 0, limit lower=0 upper=1.5708 effort=1 velocity=1
- added joint revolute_2: type continuous, parent part_1, child 9_1_gearbox_from_mas_automation, origin xyz=0 0.0185 0 rpy=3.14159 -0 3.14159, axis -0 -1 -0

File: sim/vector_description/urdf/vector.xacro (robot description, xacro)
@@ -1,616 +1,4683 @@
-<?xml version="1.0" ?>
-<robot name="vector" xmlns:xacro="http://www.ros.org/wiki/xacro">
-<xacro:arg name="ros2_controllers_config" default="config/industrial_robot_ros2_controllers.yaml" />
-<xacro:include filename="$(find vector_description)/urdf/materials.xacro" />
-<xacro:include filename="$(find vector_description)/urdf/vector.trans" />
-<xacro:include filename="$(find vector_description)/urdf/vector.gazebo" />
-<xacro:include filename="$(find vector_description)/urdf/vector.ros2_control.xacro" />
-<link name="base_link">
-  <inertial>
-    <origin xyz="0.0 0.0 -0.5" rpy="0 0 0"/>
-    <mass value="100.0"/>
-    <inertia ixx="1.0" iyy="1.0" izz="0.5" ixy="0.0" iyz="0.0" ixz="0.0"/>
-  </inertial>
-  <visual name="base_bottom_visual">
-    <origin xyz="-0.212176 -0.203 -0.0275" rpy="0 0 0"/>
-    <geometry>
-      <mesh filename="file://$(find vector_description)/meshes/base_bottomkaran.stl" scale="0.001 0.001 0.001"/>
-    </geometry>
-    <material name="grey"/>
-  </visual>
-  <visual name="base_column_visual">
-    <origin xyz="0 0 -0.0605" rpy="0 0 0"/>
-    <geometry>
-      <mesh filename="file://$(find vector_description)/meshes/base_column.stl" scale="0.0015 0.0015 0.00125"/>
-    </geometry>
-    <material name="black"/>
-  </visual>
-  <collision name="rear_caster_collision">
-    <origin xyz="-0.18 0.0 0.0195" rpy="0 0 0"/>
-    <geometry>
-      <sphere radius="0.02"/>
-    </geometry>
-  </collision>
-  <collision name="front_caster_collision">
-    <origin xyz="0.18 0.0 0.0195" rpy="0 0 0"/>
-    <geometry>
-      <sphere radius="0.02"/>
-    </geometry>
-  </collision>
-</link>
-<link name="slider_1">
-  <inertial>
-    <origin xyz="0.0 0.0 0.0" rpy="0 0 0"/>
-    <mass value="0.2"/>
-    <inertia ixx="0.001" iyy="0.001" izz="0.001" ixy="0" iyz="0" ixz="0"/>
-  </inertial>
-  <visual>
-    <origin xyz="-0.131878 -0.005317 -1.244" rpy="0 0 0"/>
-    <geometry>
-      <mesh filename="file://$(find vector_description)/meshes/slider_1.stl" scale="0.001 0.001 0.001"/>
-    </geometry>
-    <material name="black"/>
-  </visual>
-</link>
-<link name="torso_1">
-  <inertial>
-    <origin xyz="0.0 0.0 0.0" rpy="0 0 0"/>
-    <mass value="0.2"/>
-    <inertia ixx="0.001" iyy="0.001" izz="0.001" ixy="0" iyz="0" ixz="0"/>
-  </inertial>
-  <visual>
-    <origin xyz="-0.15 0.0 -0.991427" rpy="0 0 0"/>
-    <geometry>
-      <mesh filename="file://$(find vector_description)/meshes/torso_1.stl" scale="0.001 0.001 0.001"/>
-    </geometry>
-    <material name="dark_grey"/>
-  </visual>
-  <visual name="front_left_shoulder_cover">
-    <origin xyz="0.01643 0.240 0.041815" rpy="0 0 0"/>
-    <geometry>
-      <mesh filename="file://$(find vector_description)/meshes/shouldercover3.stl" scale="0.00025 0.00025 0.00025"/>
-    </geometry>
-    <material name="light_grey"/>
-  </visual>
-  <visual name="back_right_shoulder_cover">
-    <origin xyz="0.10643 -0.240 0.041815" rpy="0 0 3.14159265"/>
-    <geometry>
-      <mesh filename="file://$(find vector_description)/meshes/shouldercover3.stl" scale="0.00025 0.00025 0.00025"/>
-    </geometry>
-    <material name="light_grey"/>
-  </visual>
-</link>
-<link name="left_arm_link_1_1">
-  <inertial>
-    <origin xyz="0.0 0.0 0.0" rpy="0 0 0"/>
-    <mass value="0.2"/>
-    <inertia ixx="0.001" iyy="0.001" izz="0.001" ixy="0" iyz="0" ixz="0"/>
-  </inertial>
-  <visual>
-    <origin xyz="-0.21143 -0.13 -1.063242" rpy="0 0 0"/>
-    <geometry>
-      <mesh filename="file://$(find vector_description)/meshes/left_arm_link_1_1.stl" scale="0.001 0.001 0.001"/>
-    </geometry>
-    <material name="silver"/>
-  </visual>
-</link>
-<link name="left_shoulder_1">
-  <inertial>
-    <origin xyz="0.0 0.0 0.0" rpy="0 0 0"/>
-    <mass value="0.2"/>
-    <inertia ixx="0.001" iyy="0.001" izz="0.001" ixy="0" iyz="0" ixz="0"/>
-  </inertial>
-  <visual>
-    <origin xyz="-0.18828 -0.191 -1.063242" rpy="0 0 0"/>
-    <geometry>
-      <mesh filename="file://$(find vector_description)/meshes/left_shoulder_1.stl" scale="0.001 0.001 0.001"/>
-    </geometry>
-    <material name="silver"/>
-  </visual>
-</link>
-<link name="right_arm_link_1_1">
-  <inertial>
-    <origin xyz="0.0 0.0 0.0" rpy="0 0 0"/>
-    <mass value="0.2"/>
-    <inertia ixx="0.001" iyy="0.001" izz="0.001" ixy="0" iyz="0" ixz="0"/>
-  </inertial>
-  <visual>
-    <origin xyz="-0.21143 0.125642 -1.063242" rpy="0 0 0"/>
-    <geometry>
-      <mesh filename="file://$(find vector_description)/meshes/right_arm_link_1_1.stl" scale="0.001 0.001 0.001"/>
-    </geometry>
-    <material name="silver"/>
-  </visual>
-</link>
-<link name="right_shoulder_1">
-  <inertial>
-    <origin xyz="0.0 0.0 0.0" rpy="0 0 0"/>
-    <mass value="0.2"/>
-    <inertia ixx="0.001" iyy="0.001" izz="0.001" ixy="0" iyz="0" ixz="0"/>
-  </inertial>
-  <visual>
-    <origin xyz="-0.18828 0.186642 -1.063242" rpy="0 0 0"/>
-    <geometry>
-      <mesh filename="file://$(find vector_description)/meshes/right_shoulder_1.stl" scale="0.001 0.001 0.001"/>
-    </geometry>
-    <material name="silver"/>
-  </visual>
-</link>
-<link name="right_bicep_1">
-  <inertial>
-    <origin xyz="0.0 0.0 0.0" rpy="0 0 0"/>
-    <mass value="0.2"/>
-    <inertia ixx="0.001" iyy="0.001" izz="0.001" ixy="0" iyz="0" ixz="0"/>
-  </inertial>
-  <visual>
-    <origin xyz="-0.21143 0.186998 -1.014718" rpy="0 0 0"/>
-    <geometry>
-      <mesh filename="file://$(find vector_description)/meshes/right_bicep_1.stl" scale="0.001 0.001 0.001"/>
-    </geometry>
-    <material name="silver"/>
-  </visual>
-  <collision>
-    <origin xyz="-0.21143 0.186998 -1.014718" rpy="0 0 0"/>
-    <geometry>
-      <mesh filename="file://$(find vector_description)/meshes/right_bicep_1.stl" scale="0.001 0.001 0.001"/>
-    </geometry>
-  </collision>
-</link>
-<link name="left_bicep_1">
-  <inertial>
-    <origin xyz="0.0 0.0 0.0" rpy="0 0 0"/>
-    <mass value="0.2"/>
-    <inertia ixx="0.001" iyy="0.001" izz="0.001" ixy="0" iyz="0" ixz="0"/>
-  </inertial>
-  <visual>
-    <origin xyz="-0.21143 -0.191 -1.010242" rpy="0 0 0"/>
-    <geometry>
-      <mesh filename="file://$(find vector_description)/meshes/left_bicep_1.stl" scale="0.001 0.001 0.001"/>
-    </geometry>
-    <material name="silver"/>
-  </visual>
-  <collision>
-    <origin xyz="-0.21143 -0.191 -1.010242" rpy="0 0 0"/>
-    <geometry>
-      <mesh filename="file://$(find vector_description)/meshes/left_bicep_1.stl" scale="0.001 0.001 0.001"/>
-    </geometry>
-  </collision>
-</link>
-<link name="right_forearm_v1_1">
-  <inertial>
-    <origin xyz="0.0 0.0 0.0" rpy="0 0 0"/>
-    <mass value="0.2"/>
-    <inertia ixx="0.001" iyy="0.001" izz="0.001" ixy="0" iyz="0" ixz="0"/>
-  </inertial>
-  <visual>
-    <origin xyz="-0.233013 0.217698 -0.781318" rpy="0 0 0"/>
-    <geometry>
-      <mesh filename="file://$(find vector_description)/meshes/right_forearm_v1_1.stl" scale="0.001 0.001 0.001"/>
-    </geometry>
-    <material name="silver"/>
-  </visual>
-  <collision>
-    <origin xyz="-0.233013 0.217698 -0.781318" rpy="0 0 0"/>
-    <geometry>
-      <mesh filename="file://$(find vector_description)/meshes/right_forearm_v1_1.stl" scale="0.001 0.001 0.001"/>
-    </geometry>
-  </collision>
-</link>
-<link name="left_forearm_v2_1">
-  <inertial>
-    <origin xyz="0.0 0.0 0.0" rpy="0 0 0"/>
-    <mass value="0.2"/>
-    <inertia ixx="0.001" iyy="0.001" izz="0.001" ixy="0" iyz="0" ixz="0"/>
-  </inertial>
-  <visual>
-    <origin xyz="-0.233013 -0.1603 -0.776842" rpy="0 0 0"/>
-    <geometry>
-      <mesh filename="file://$(find vector_description)/meshes/left_forearm_v2_1.stl" scale="0.001 0.001 0.001"/>
-    </geometry>
-    <material name="silver"/>
-  </visual>
-  <collision>
-    <origin xyz="-0.233013 -0.1603 -0.776842" rpy="0 0 0"/>
-    <geometry>
-      <mesh filename="file://$(find vector_description)/meshes/left_forearm_v2_1.stl" scale="0.001 0.001 0.001"/>
-    </geometry>
-  </collision>
-</link>
-<link name="neck_v2_1">
-  <inertial>
-    <origin xyz="0.0 0.0 0.0" rpy="0 0 0"/>
-    <mass value="0.2"/>
-    <inertia ixx="0.001" iyy="0.001" izz="0.001" ixy="0" iyz="0" ixz="0"/>
-  </inertial>
-  <visual>
-    <origin xyz="-0.223 -0.022179 -1.142427" rpy="0 0 0"/>
-    <geometry>
-      <mesh filename="file://$(find vector_description)/meshes/neck_v2_1.stl" scale="0.001 0.001 0.001"/>
-    </geometry>
-    <material name="black"/>
-  </visual>
-</link>
-<link name="head_v1_1">
-  <inertial>
-    <origin xyz="0.0 0.0 0.0" rpy="0 0 0"/>
-    <mass value="0.2"/>
-    <inertia ixx="0.001" iyy="0.001" izz="0.001" ixy="0" iyz="0" ixz="0"/>
-  </inertial>
-  <visual>
-    <origin xyz="-0.223 -0.002179 -1.165427" rpy="0 0 0"/>
-    <geometry>
-      <mesh filename="file://$(find vector_description)/meshes/head_v1_1.stl" scale="0.001 0.001 0.001"/>
-    </geometry>
-    <material name="silver"/>
-  </visual>
-</link>
-<!-- INSERT THIS FOR NEW GAZEBO ENGINE OVERRIDES -->
-<gazebo reference="head_v1_1">
-  <visual>
-    <material>
-      <ambient>1 1 1 0</ambient>
-      <diffuse>1 1 1 0</diffuse>
-      <specular>0 0 0 0</specular>
-      <emissive>0 0 0 0</emissive>
-    </material>
-  </visual>
-</gazebo>
-<link name="livox_mid360_link">
-  <inertial>
-    <origin xyz="0.0 0.0 0.0" rpy="0 0 0"/>
-    <mass value="0.265"/>
-    <inertia ixx="0.0002" iyy="0.0002" izz="0.0003" ixy="0" iyz="0" ixz="0"/>
-  </inertial>
-  <visual name="livox_mid360_visual">
-    <origin xyz="0 0 0" rpy="0 0 0"/>
-    <geometry>
-      <cylinder radius="0.053" length="0.052"/>
-    </geometry>
-    <material name="dark_grey"/>
-  </visual>
-</link>
-<joint name="livox_mid360_joint" type="fixed">
-  <!-- Mounted on top of the base column, just below the slider mechanism.
-       slider_1 origin is at (0.131878, 0.005317, 1.244) from base_link,
-       so we offset back to center the LiDAR on the column axis. -->
-  <origin xyz="-0.131878 -0.005317 -0.01" rpy="0 0 0"/>
-  <parent link="slider_1"/>
-  <child link="livox_mid360_link"/>
-</joint>
-<link name="right_wheel_1">
-  <inertial>
-    <origin xyz="-2.7445143105647544e-17 -0.01999999999999988 -1.3877787807814457e-17" rpy="0 0 0"/>
-    <mass value="1.168672467135403"/>
-    <inertia ixx="0.003078" iyy="0.005843" izz="0.003078" ixy="0.0" iyz="0.0" ixz="-0.0"/>
-  </inertial>
-  <visual>
-    <origin xyz="-0.0 0.203 -0.0725" rpy="0 0 0"/>
-    <geometry>
-      <mesh filename="file://$(find vector_description)/meshes/right_wheel_1.stl" scale="0.001 0.001 0.001"/>
-    </geometry>
-    <material name="black"/>
-  </visual>
-  <collision>
-    <origin xyz="0 0 0" rpy="1.5707963 0 0"/>
-    <geometry>
-      <cylinder radius="0.075" length="0.08"/>
-    </geometry>
-  </collision>
-</link>
-<link name="left_wheel_1">
-  <inertial>
-    <origin xyz="6.228708332783829e-17 0.01999999999999988 0.0" rpy="0 0 0"/>
-    <mass value="1.168672467135403"/>
-    <inertia ixx="0.003078" iyy="0.005843" izz="0.003078" ixy="0.0" iyz="0.0" ixz="-0.0"/>
-  </inertial>
-  <visual>
-    <origin xyz="-0.0 -0.203 -0.0725" rpy="0 0 0"/>
-    <geometry>
-      <mesh filename="file://$(find vector_description)/meshes/left_wheel_1.stl" scale="0.001 0.001 0.001"/>
-    </geometry>
-    <material name="black"/>
-  </visual>
-  <collision>
-    <origin xyz="0 0 0" rpy="1.5707963 0 0"/>
-    <geometry>
-      <cylinder radius="0.075" length="0.08"/>
-    </geometry>
-  </collision>
-</link>
-<link name="camera_1">
-  <inertial>
-    <origin xyz="0.0 0.0 0.0" rpy="0 0 0"/>
-    <mass value="0.2"/>
-    <inertia ixx="0.001" iyy="0.001" izz="0.001" ixy="0" iyz="0" ixz="0"/>
-  </inertial>
-  <visual>
-    <origin xyz="-0.268 -0.003429 -1.227137" rpy="0 0 0"/>
-    <geometry>
-      <mesh filename="file://$(find vector_description)/meshes/camera_1.stl" scale="0.001 0.001 0.001"/>
-    </geometry>
-    <material name="black"/>
-  </visual>
-</link>
-<link name="left_hand_palm_1">
-  <inertial>
-    <origin xyz="0.0 0.0 0.0" rpy="0 0 0"/>
-    <mass value="0.2"/>
-    <inertia ixx="0.001" iyy="0.001" izz="0.001" ixy="0" iyz="0" ixz="0"/>
-  </inertial>
-  <visual>
-    <origin xyz="-0.48 -0.18 -0.8" rpy="0 0 0"/>
-    <geometry>
-      <mesh filename="file://$(find vector_description)/meshes/left_hand_palm_1.stl" scale="0.001 0.001 0.001"/>
-    </geometry>
-    <material name="dark_grey"/>
-  </visual>
-</link>
-<link name="left_hand_finger_1">
-  <inertial>
-    <origin xyz="0.0 0.0 0.0" rpy="0 0 0"/>
-    <mass value="0.2"/>
-    <inertia ixx="0.001" iyy="0.001" izz="0.001" ixy="0" iyz="0" ixz="0"/>
-  </inertial>
-  <visual>
-    <origin xyz="-0.552276 -0.2 -0.816596" rpy="0 0 0"/>
-    <geometry>
-      <mesh filename="file://$(find vector_description)/meshes/left_hand_finger_1.stl" scale="0.001 0.001 0.001"/>
-    </geometry>
-    <material name="silver"/>
-  </visual>
-</link>
-<link name="right_hand_palm_1">
-  <inertial>
-    <origin xyz="0.0 0.0 0.0" rpy="0 0 0"/>
-    <mass value="0.2"/>
-    <inertia ixx="0.001" iyy="0.001" izz="0.001" ixy="0" iyz="0" ixz="0"/>
-  </inertial>
-  <visual>
-    <origin xyz="-0.482 0.177 -0.79" rpy="0 0 0"/>
-    <geometry>
-      <mesh filename="file://$(find vector_description)/meshes/right_hand_palm_1.stl" scale="0.001 0.001 0.001"/>
-    </geometry>
-    <material name="dark_grey"/>
-  </visual>
-</link>
-<link name="right_hand_finger_1">
-  <inertial>
-    <origin xyz="0.0 0.0 0.0" rpy="0 0 0"/>
-    <mass value="0.2"/>
-    <inertia ixx="0.001" iyy="0.001" izz="0.001" ixy="0" iyz="0" ixz="0"/>
-  </inertial>
-  <visual>
-    <origin xyz="-0.552087 0.195998 -0.763566" rpy="0 0 0"/>
-    <geometry>
-      <mesh filename="file://$(find vector_description)/meshes/right_hand_finger_1.stl" scale="0.001 0.001 0.001"/>
-    </geometry>
-    <material name="silver"/>
-  </visual>
-</link>
-<joint name="slider_z_axis" type="prismatic">
-  <origin xyz="0.131878 0.005317 1.244" rpy="0 0 0"/>
-  <parent link="base_link"/>
-  <child link="slider_1"/>
-  <axis xyz="0.0 0.0 1.0"/>
-  <limit upper="0.4" lower="-0.6" effort="2000" velocity="100"/>
-  <dynamics damping="50.0" friction="10.0"/>
-</joint>
-<joint name="torso_with_slider" type="fixed">
-  <origin xyz="0.018122 -0.005317 -0.252573" rpy="0 0 0"/>
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