Commit message: refactor(sim): update vector robot kinematics, inertials, and Gazebo controllers
- Correct joint origins and mass inertials in URDF (vector.xacro) to fix forward tilt instability.
- Update joint_trajectory_controller active joints configuration.
- Adjust spawn position, yaw orientation, and controller startup in launch file.
- Update torso PID gains, limits, and gravity feedforward to match 31.62kg robot mass.
- Map updated joint names in torso safety guard.

File: sim/vector_description/urdf/vector.ros2_control.xacro (robot description, xacro)
@@ -5,5 +5,27 @@
       <plugin>gz_ros2_control/GazeboSimSystem</plugin>
     </hardware>
-    <joint name="revolute_1">
+    <joint name="left_wheel_joint">
+      <command_interface name="velocity"/>
+      <state_interface name="position">
+        <param name="initial_value">0.0</param>
+      </state_interface>
+      <state_interface name="velocity"/>
+    </joint>
+    <joint name="right_wheel_joint">
+      <command_interface name="velocity"/>
+      <state_interface name="position">
+        <param name="initial_value">0.0</param>
+      </state_interface>
+      <state_interface name="velocity"/>
+    </joint>
+    <joint name="torso_joint">
+      <command_interface name="effort"/>
+      <state_interface name="position">
+        <param name="initial_value">0.39</param>
+      </state_interface>
+      <state_interface name="velocity"/>
+      <state_interface name="effort"/>
+    </joint>
+    <joint name="shoulder_link_1">
       <command_interface name="position"/>
       <state_interface name="position">
@@ -12,5 +34,61 @@
       <state_interface name="velocity"/>
     </joint>
-    <joint name="revolute_2">
+    <joint name="left_shoulder">
+      <command_interface name="position"/>
+      <state_interface name="position">
+        <param name="initial_value">0.0</param>
+      </state_interface>
+      <state_interface name="velocity"/>
+    </joint>
+    <joint name="left_bicep">
+      <command_interface name="position"/>
+      <state_interface name="position">
+        <param name="initial_value">0.0</param>
+      </state_interface>
+      <state_interface name="velocity"/>
+    </joint>
+    <joint name="left_forearm">
+      <command_interface name="position"/>
+      <state_interface name="position">
+        <param name="initial_value">0.0</param>
+      </state_interface>
+      <state_interface name="velocity"/>
+    </joint>
+    <joint name="right_shoulder_1">
+      <command_interface name="position"/>
+      <state_interface name="position">
+        <param name="initial_value">0.0</param>
+      </state_interface>
+      <state_interface name="velocity"/>
+    </joint>
+    <joint name="right_shoulder_2">
+      <command_interface name="position"/>
+      <state_interface name="position">
+        <param name="initial_value">0.0</param>
+      </state_interface>
+      <state_interface name="velocity"/>
+    </joint>
+    <joint name="right_bicep">
+      <command_interface name="position"/>
+      <state_interface name="position">
+        <param name="initial_value">0.0</param>
+      </state_interface>
+      <state_interface name="velocity"/>
+    </joint>
+    <joint name="right_forearm">
+      <command_interface name="position"/>
+      <state_interface name="position">
+        <param name="initial_value">0.0</param>
+      </state_interface>
+      <state_interface name="velocity"/>
+    </joint>
+    <joint name="right_wrist_1">
+      <command_interface name="position"/>
+      <state_interface name="position">
+        <param name="initial_value">0.0</param>
+      </state_interface>
+      <state_interface name="velocity"/>
+    </joint>
+    <joint name="right_wrist_2">
       <command_interface name="position"/>
       <state_interface name="position">

File: sim/vector_description/urdf/vector.xacro (robot description, xacro)
@@ -33,5 +33,5 @@
         </visual>
     <collision><origin xyz="0.0 -0.0087 0.0" rpy="0 0 0" /><geometry><box size="0.078 0.1275 0.078" /></geometry></collision></link>
-    <link name="part_1">
+    <link name="right_wheel_link">
         <inertial>
             <mass value="0.795632" />
@@ -48,6 +48,6 @@
             </material>
         </visual>
-    <collision><origin xyz="0.0 0.0 0.0" rpy="0 0 0" /><geometry><box size="0.1524 0.037 0.1524" /></geometry></collision></link>
-    <link name="part_1_1">
+    <collision><origin xyz="0.0 0.0 0.0" rpy="1.5708 0 0" /><geometry><cylinder radius="0.0762" length="0.037" /></geometry></collision></link>
+    <link name="left_wheel_link">
         <inertial>
             <mass value="0.795632" />
@@ -64,6 +64,11 @@
             </material>
         </visual>
-    <collision><origin xyz="0.0 0.0185 0.0" rpy="0 0 0" /><geometry><box size="0.1524 0.037 0.1524" /></geometry></collision></link>
-    <link name="root">
+    <collision><origin xyz="0.0 0.0185 0.0" rpy="1.5708 0 0" /><geometry><cylinder radius="0.0762" length="0.037" /></geometry></collision></link>
+        <link name="base_link">
+        <inertial>
+            <mass value="66.476139" />
+            <origin xyz="0.049547 -0.005405 0.025724" rpy="0 0 0" />
+            <inertia ixx="5.079439634e+00" ixy="-2.193859608e-02" ixz="-1.312023858e-01" iyy="4.725292650e+00" iyz="5.987075030e-01" izz="2.926682437e+00" />
+        </inertial>
         <visual>
             <origin xyz="0.219836 0.157455 0.0584722" rpy="2.92124e-16 6.245e-17 1.5708" />
@@ -2495,6 +2500,25 @@
             </material>
         </visual>
-        <visual>
-            <origin xyz="0.034824 0.121366 0.966282" rpy="-3.23522e-16 -6.12323e-17 3.14159" />
+        <collision>
+            <origin xyz="0.0488 0.0656 0.2" rpy="0 0 0" />
+            <geometry>
+                <box size="0.6762 0.6624 0.4" />
+            </geometry>
+        </collision>
+    </link>
+    <link name="torso_link">
+        <inertial>
+            <mass value="12.265738" />
+            <origin xyz="-0.107959 0.054868 0.006976" rpy="0 0 0" />
+            <inertia ixx="9.196184751e-02" ixy="7.723493482e-03" ixz="2.212420539e-03" iyy="1.552825481e-01" iyz="5.903978641e-04" izz="1.402793003e-01" />
+        </inertial>
+        <collision>
+            <origin xyz="-0.101200 0.065600 -0.041427" rpy="0 0 0" />
+            <geometry>
+                <box size="0.6762 0.6624 1.45" />
+            </geometry>
+        </collision>
+<visual>
+            <origin xyz="-0.115176 0.121366 -0.025145" rpy="-3.23522e-16 -6.12323e-17 3.14159" />
             <geometry>
                 <mesh filename="file://$(find vector_description)/meshes/Speaker_1_box.stl" scale="1 1 1" />
@@ -2505,6 +2529,6 @@
             </material>
         </visual>
-        <visual>
-            <origin xyz="0.084824 0.0513664 0.937501" rpy="1.5708 -6.12323e-17 3.14159" />
+<visual>
+            <origin xyz="-0.065176 0.051366 -0.053926" rpy="1.5708 -6.12323e-17 3.14159" />
             <geometry>
                 <mesh filename="file://$(find vector_description)/meshes/Part_3_Mirrored.stl" scale="1 1 1" />
@@ -2515,6 +2539,6 @@
             </material>
         </visual>
-        <visual>
-            <origin xyz="0.184824 0.0517664 0.917101" rpy="0 -1.5708 4.78784e-16" />
+<visual>
+            <origin xyz="0.034824 0.051766 -0.074326" rpy="0 -1.5708 4.78784e-16" />
             <geometry>
                 <mesh filename="file://$(find vector_description)/meshes/Part_3_Mirrored_Mirrored.stl" scale="1 1 1" />
@@ -2525,6 +2549,6 @@
             </material>
         </visual>
-        <visual>
-            <origin xyz="0.00522396 0.151366 0.902101" rpy="5.38978e-16 -1.18329e-30 -1.5708" />
+<visual>
+            <origin xyz="-0.144776 0.151366 -0.089326" rpy="5.38978e-16 -1.18329e-30 -1.5708" />
             <geometry>
                 <mesh filename="file://$(find vector_description)/meshes/Part_3_1.stl" scale="1 1 1" />
@@ -2535,6 +2559,6 @@
             </material>
         </visual>
-        <visual>
-            <origin xyz="0.034824 -0.0206336 0.975601" rpy="1.97215e-30 -6.12323e-17 3.14159" />
+<visual>
+            <origin xyz="-0.115176 -0.020634 -0.015826" rpy="1.97215e-30 -6.12323e-17 3.14159" />
             <geometry>
                 <mesh filename="file://$(find vector_description)/meshes/Back_top_plate.stl" scale="1 1 1" />
@@ -2545,6 +2569,6 @@
             </material>
         </visual>
-        <visual>
-            <origin xyz="0.084824 0.0509664 1.0171" rpy="1.40939e-30 -6.12323e-17 3.14159" />
+<visual>
+            <origin xyz="-0.065176 0.050966 0.025673" rpy="1.40939e-30 -6.12323e-17 3.14159" />
             <geometry>
                 <mesh filename="file://$(find vector_description)/meshes/Part_3_1.stl" scale="1 1 1" />
@@ -2555,6 +2579,6 @@
             </material>
         </visual>
-        <visual>
-            <origin xyz="0.184824 0.0509664 1.0171" rpy="1.40939e-30 -6.12323e-17 3.14159" />
+<visual>
+            <origin xyz="0.034824 0.050966 0.025673" rpy="1.40939e-30 -6.12323e-17 3.14159" />
             <geometry>
                 <mesh filename="file://$(find vector_description)/meshes/Part_3_1.stl" scale="1 1 1" />
@@ -2565,6 +2589,6 @@
             </material>
         </visual>
-        <visual>
-            <origin xyz="0.034824 0.0513664 0.887101" rpy="1.97215e-30 -6.12323e-17 3.14159" />
+<visual>
+            <origin xyz="-0.115176 0.051366 -0.104326" rpy="1.97215e-30 -6.12323e-17 3.14159" />
             <geometry>
                 <mesh filename="file://$(find vector_description)/meshes/Part_17_2.stl" scale="1 1 1" />
@@ -2575,6 +2599,6 @@
             </material>
         </visual>
-        <visual>
-            <origin xyz="-0.115176 0.0517664 0.917101" rpy="0 -1.5708 -4.3715e-16" />
+<visual>
+            <origin xyz="-0.265176 0.051766 -0.074326" rpy="0 -1.5708 -4.3715e-16" />
             <geometry>
                 <mesh filename="file://$(find vector_description)/meshes/Part_3_Mirrored.stl" scale="1 1 1" />
@@ -2585,6 +2609,6 @@
             </material>
         </visual>
-        <visual>
-            <origin xyz="0.034824 0.0513664 0.887101" rpy="1.97215e-30 -6.12323e-17 3.14159" />
+<visual>
+            <origin xyz="-0.115176 0.051366 -0.104326" rpy="1.97215e-30 -6.12323e-17 3.14159" />
             <geometry>
                 <mesh filename="file://$(find vector_description)/meshes/Part_12_3.stl" scale="1 1 1" />
@@ -2595,6 +2619,6 @@
             </material>
         </visual>
-        <visual>
-            <origin xyz="0.064424 0.151366 0.902101" rpy="3.14159 -2.71171e-30 -1.5708" />
+<visual>
+            <origin xyz="-0.085576 0.151366 -0.089326" rpy="3.14159 -2.71171e-30 -1.5708" />
             <geometry>
                 <mesh filename="file://$(find vector_description)/meshes/Part_3_Mirrored.stl" scale="1 1 1" />
@@ -2605,6 +2629,6 @@
             </material>
         </visual>
-        <visual>
-            <origin xyz="0.00482396 0.0509664 1.0371" rpy="0 1.5708 3.14159" />
+<visual>
+            <origin xyz="-0.145176 0.050966 0.045673" rpy="0 1.5708 3.14159" />
             <geometry>
                 <mesh filename="file://$(find vector_description)/meshes/Part_3_3.stl" scale="1 1 1" />
@@ -2615,6 +2639,6 @@
             </material>
         </visual>
-        <visual>
-            <origin xyz="0.034824 0.0513664 0.887101" rpy="1.97215e-30 -6.12323e-17 3.14159" />
+<visual>
+            <origin xyz="-0.115176 0.051366 -0.104326" rpy="1.97215e-30 -6.12323e-17 3.14159" />
             <geometry>
                 <mesh filename="file://$(find vector_description)/meshes/Part_8_2.stl" scale="1 1 1" />
@@ -2625,6 +2649,6 @@
             </material>
         </visual>
-        <visual>
-            <origin xyz="0.00522396 -0.0686336 1.0371" rpy="0 1.5708 -1.5708" />
+<visual>
+            <origin xyz="-0.144776 -0.068634 0.045673" rpy="0 1.5708 -1.5708" />
             <geometry>
                 <mesh filename="file://$(find vector_description)/meshes/Part_3_Mirrored_1.stl" scale="1 1 1" />
@@ -2635,6 +2659,6 @@
             </material>
         </visual>
-        <visual>
-            <origin xyz="0.064424 -0.0686336 1.0371" rpy="0 1.5708 -4.71239" />
+<visual>
+            <origin xyz="-0.085576 -0.068634 0.045673" rpy="0 1.5708 -4.71239" />
             <geometry>
                 <mesh filename="file://$(find vector_description)/meshes/Part_3_Mirrored_Mirrored_1.stl" scale="1 1 1" />
@@ -2645,6 +2669,6 @@
             </material>
         </visual>
-        <visual>
-            <origin xyz="0.184824 0.0517664 1.0171" rpy="-3.14159 -6.12323e-17 3.14159" />
+<visual>
+            <origin xyz="0.034824 0.051766 0.025673" rpy="-3.14159 -6.12323e-17 3.14159" />
             <geometry>
                 <mesh filename="file://$(find vector_description)/meshes/Part_3_Mirrored.stl" scale="1 1 1" />
@@ -2655,6 +2679,6 @@
             </material>
         </visual>
-        <visual>
-            <origin xyz="0.00522396 0.151366 1.0171" rpy="-6.12323e-17 -2.34809e-30 -1.5708" />
+<visual>
+            <origin xyz="-0.144776 0.151366 0.025673" rpy="-6.12323e-17 -2.34809e-30 -1.5708" />
             <geometry>
                 <mesh filename="file://$(find vector_description)/meshes/Part_3_1.stl" scale="1 1 1" />
@@ -2665,6 +2689,6 @@
             </material>
         </visual>
-        <visual>
-            <origin xyz="0.034824 0.0513664 0.887101" rpy="1.97215e-30 -6.12323e-17 3.14159" />
+<visual>
+            <origin xyz="-0.115176 0.051366 -0.104326" rpy="1.97215e-30 -6.12323e-17 3.14159" />
             <geometry>
                 <mesh filename="file://$(find vector_description)/meshes/Part_9_2.stl" scale="1 1 1" />
@@ -2675,6 +2699,6 @@
             </material>
         </visual>
-        <visual>
-            <origin xyz="0.035574 0.173666 0.9503" rpy="1.03062e-17 -3.11033e-16 3.14159" />
+<visual>
+            <origin xyz="-0.114426 0.173666 -0.041127" rpy="1.03062e-17 -3.11033e-16 3.14159" />
             <geometry>
                 <mesh filename="file://$(find vector_description)/meshes/Torso_front_shield.stl" scale="1 1 1" />
@@ -2685,6 +2709,6 @@
             </material>
         </visual>
-        <visual>
-            <origin xyz="0.034824 0.0513664 0.887101" rpy="1.97215e-30 -6.12323e-17 3.14159" />
+<visual>
+            <origin xyz="-0.115176 0.051366 -0.104326" rpy="1.97215e-30 -6.12323e-17 3.14159" />
             <geometry>
                 <mesh filename="file://$(find vector_description)/meshes/Part_7_2.stl" scale="1 1 1" />
@@ -2695,6 +2719,6 @@
             </material>
         </visual>
-        <visual>
-            <origin xyz="-0.115176 0.0509664 0.917101" rpy="0 -1.5708 3.14159" />
+<visual>
+            <origin xyz="-0.265176 0.050966 -0.074326" rpy="0 -1.5708 3.14159" />
             <geometry>
                 <mesh filename="file://$(find vector_description)/meshes/Part_3_1.stl" scale="1 1 1" />
@@ -2705,6 +2729,6 @@
             </material>
         </visual>
-        <visual>
-            <origin xyz="0.034824 0.0513664 0.887101" rpy="1.97215e-30 -6.12323e-17 3.14159" />
+<visual>
+            <origin xyz="-0.115176 0.051366 -0.104326" rpy="1.97215e-30 -6.12323e-17 3.14159" />
             <geometry>
                 <mesh filename="file://$(find vector_description)/meshes/Part_2_3.stl" scale="1 1 1" />
@@ -2715,6 +2739,6 @@
             </material>
         </visual>
-        <visual>
-            <origin xyz="0.034824 0.0513664 0.887101" rpy="1.97215e-30 -6.12323e-17 3.14159" />
+<visual>
+            <origin xyz="-0.115176 0.051366 -0.104326" rpy="1.97215e-30 -6.12323e-17 3.14159" />
             <geometry>
                 <mesh filename="file://$(find vector_description)/meshes/Part_6_2.stl" scale="1 1 1" />
@@ -2725,6 +2749,6 @@
             </material>
         </visual>
-        <visual>
-            <origin xyz="0.034824 0.0513664 0.866101" rpy="-3.23522e-16 -6.12323e-17 3.14159" />
+<visual>
+            <origin xyz="-0.115176 0.051366 -0.125326" rpy="-3.23522e-16 -6.12323e-17 3.14159" />
             <geometry>
                 <mesh filename="file://$(find vector_description)/meshes/extra_2xMS_2mm_Base_Plate.stl" scale="1 1 1" />
@@ -2735,6 +2759,6 @@
             </material>
         </visual>
-        <visual>
-            <origin xyz="0.064424 0.151366 1.0171" rpy="3.14159 -1.9475e-30 -1.5708" />
+<visual>
+            <origin xyz="-0.085576 0.151366 0.025673" rpy="3.14159 -1.9475e-30 -1.5708" />
             <geometry>
                 <mesh filename="file://$(find vector_description)/meshes/Part_3_Mirrored.stl" scale="1 1 1" />
@@ -2745,6 +2769,6 @@
             </material>
         </visual>
-        <visual>
-            <origin xyz="0.084824 0.0513664 0.937501" rpy="1.5708 -6.12323e-17 3.14159" />
+<visual>
+            <origin xyz="-0.065176 0.051366 -0.053926" rpy="1.5708 -6.12323e-17 3.14159" />
             <geometry>
                 <mesh filename="file://$(find vector_description)/meshes/Part_3_1.stl" scale="1 1 1" />
@@ -2755,6 +2779,6 @@
             </material>
         </visual>
-        <visual>
-            <origin xyz="0.034824 0.0513664 0.887101" rpy="1.97215e-30 -6.12323e-17 3.14159" />
+<visual>
+            <origin xyz="-0.115176 0.051366 -0.104326" rpy="1.97215e-30 -6.12323e-17 3.14159" />
             <geometry>
                 <mesh filename="file://$(find vector_description)/meshes/Part_3_4.stl" scale="1 1 1" />
@@ -2765,6 +2789,6 @@
             </material>
         </visual>
-        <visual>
-            <origin xyz="0.034824 0.0513664 0.887101" rpy="1.97215e-30 -6.12323e-17 3.14159" />
+<visual>
+            <origin xyz="-0.115176 0.051366 -0.104326" rpy="1.97215e-30 -6.12323e-17 3.14159" />
             <geometry>
                 <mesh filename="file://$(find vector_description)/meshes/Part_11_2.stl" scale="1 1 1" />
@@ -2775,6 +2799,6 @@
             </material>
         </visual>
-        <visual>
-            <origin xyz="0.064824 0.0517664 1.0371" rpy="0 1.5708 4.78784e-16" />
+<visual>
+            <origin xyz="-0.085176 0.051766 0.045673" rpy="0 1.5708 4.78784e-16" />
             <geometry>
                 <mesh filename="file://$(find vector_description)/meshes/Part_3_Mirrored_Mirrored_1.stl" scale="1 1 1" />
@@ -2785,6 +2809,6 @@
             </material>
         </visual>
-        <visual>
-            <origin xyz="0.034824 0.0513664 0.887101" rpy="1.97215e-30 -6.12323e-17 3.14159" />
+<visual>
+            <origin xyz="-0.115176 0.051366 -0.104326" rpy="1.97215e-30 -6.12323e-17 3.14159" />
             <geometry>
                 <mesh filename="file://$(find vector_description)/meshes/Part_16_2.stl" scale="1 1 1" />
@@ -2795,6 +2819,6 @@
             </material>
         </visual>
-        <visual>
-            <origin xyz="0.184824 0.0509664 0.917101" rpy="0 -1.5708 3.14159" />
+<visual>
+            <origin xyz="0.034824 0.050966 -0.074326" rpy="0 -1.5708 3.14159" />
             <geometry>
                 <mesh filename="file://$(find vector_description)/meshes/Part_3_Mirrored.stl" scale="1 1 1" />
@@ -2805,6 +2829,6 @@
             </material>
         </visual>
-        <visual>
-            <origin xyz="0.00522396 0.0513664 0.917101" rpy="0 -1.5708 -1.5708" />
+<visual>
+            <origin xyz="-0.144776 0.051366 -0.074326" rpy="0 -1.5708 -1.5708" />
             <geometry>
                 <mesh filename="file://$(find vector_description)/meshes/Part_3_Mirrored.stl" scale="1 1 1" />
@@ -2815,6 +2839,6 @@
             </material>
         </visual>
-        <visual>
-            <origin xyz="0.034824 0.123866 0.992101" rpy="1.97215e-30 -6.12323e-17 3.14159" />
+<visual>
+            <origin xyz="-0.115176 0.123866 0.000674" rpy="1.97215e-30 -6.12323e-17 3.14159" />
             <geometry>
                 <mesh filename="file://$(find vector_description)/meshes/_3dprinted_Front_plate.stl" scale="1 1 1" />
@@ -2825,6 +2849,6 @@
             </material>
         </visual>
-        <visual>
-            <origin xyz="0.034824 0.0513664 0.887101" rpy="1.97215e-30 -6.12323e-17 3.14159" />
+<visual>
+            <origin xyz="-0.115176 0.051366 -0.104326" rpy="1.97215e-30 -6.12323e-17 3.14159" />
             <geometry>
                 <mesh filename="file://$(find vector_description)/meshes/Part_4_3.stl" scale="1 1 1" />
@@ -2835,6 +2859,6 @@
             </material>
         </visual>
-        <visual>
-            <origin xyz="0.034824 0.0513664 0.887101" rpy="1.97215e-30 -6.12323e-17 3.14159" />
+<visual>
+            <origin xyz="-0.115176 0.051366 -0.104326" rpy="1.97215e-30 -6.12323e-17 3.14159" />
             <geometry>
                 <mesh filename="file://$(find vector_description)/meshes/Part_10_2.stl" scale="1 1 1" />
@@ -2845,6 +2869,6 @@
             </material>
         </visual>
-        <visual>
-            <origin xyz="0.00482396 0.0517664 1.0371" rpy="0 1.5708 -4.3715e-16" />
+<visual>
+            <origin xyz="-0.145176 0.051766 0.045673" rpy="0 1.5708 -4.3715e-16" />
             <geometry>
                 <mesh filename="file://$(find vector_description)/meshes/Part_3_Mirrored_1.stl" scale="1 1 1" />
@@ -2855,6 +2879,6 @@
             </material>
         </visual>
-        <visual>
-            <origin xyz="0.034824 0.0513664 0.887101" rpy="1.97215e-30 -6.12323e-17 3.14159" />
+<visual>
+            <origin xyz="-0.115176 0.051366 -0.104326" rpy="1.97215e-30 -6.12323e-17 3.14159" />
             <geometry>
                 <mesh filename="file://$(find vector_description)/meshes/Part_13_2.stl" scale="1 1 1" />
@@ -2865,6 +2889,6 @@
             </material>
         </visual>
-        <visual>
-            <origin xyz="0.084824 0.0517664 1.0171" rpy="-3.14159 -6.12323e-17 3.14159" />
+<visual>
+            <origin xyz="-0.065176 0.051766 0.025673" rpy="-3.14159 -6.12323e-17 3.14159" />
             <geometry>
                 <mesh filename="file://$(find vector_description)/meshes/Part_3_Mirrored.stl" scale="1 1 1" />
@@ -2875,6 +2899,6 @@
             </material>
         </visual>
-        <visual>
-            <origin xyz="0.034824 0.0513664 1.0857" rpy="7.92292e-16 4.8785e-17 3.14159" />
+<visual>
+            <origin xyz="-0.115176 0.051366 0.094273" rpy="7.92292e-16 4.8785e-17 3.14159" />
             <geometry>
                 <mesh filename="file://$(find vector_description)/meshes/Part_1_7.stl" scale="1 1 1" />
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