Commit message: split the base_link

File: sim/vector_description/urdf/materials.xacro (robot description, xacro)
@@ -10,4 +10,7 @@
   <color rgba="0.200 0.200 0.200 1.000"/>
 </material>
+<material name="grey">
+  <color rgba="0.500 0.500 0.500 1.000"/>
+</material>
 <material name="black">
   <color rgba="0.0 0.0 0.0 1.000"/>

File: sim/vector_description/urdf/vector.xacro (robot description, xacro)
@@ -1,6 +1,4 @@
 <?xml version="1.0" ?>
 <robot name="vector" xmlns:xacro="http://www.ros.org/wiki/xacro">
-<!-- Define xacro property for ros2_controllers config file path -->
-<!-- This allows the launch file to pass in the correct absolute path for Gazebo Harmonic -->
 <xacro:arg name="ros2_controllers_config" default="config/industrial_robot_ros2_controllers.yaml" />
 <xacro:include filename="$(find vector_description)/urdf/materials.xacro" />
@@ -9,8 +7,4 @@
 <xacro:include filename="$(find vector_description)/urdf/vector.ros2_control.xacro" />
 <link name="base_link">
-  <!-- SIM-TUNED: Light base (5 kg) at z=0.  Upper-body links are set to
-       near-zero mass (0.01 kg each) so gravity exerts almost no torque on
-       the top-heavy structure.  No collision on base_link — only wheels
-       and casters touch the ground. -->
   <inertial>
     <origin xyz="0.0 0.0 -0.5" rpy="0 0 0"/>
@@ -18,13 +12,18 @@
     <inertia ixx="1.0" iyy="1.0" izz="0.5" ixy="0.0" iyz="0.0" ixz="0.0"/>
   </inertial>
-  <visual>
+  <visual name="base_bottom_visual">
     <origin xyz="0 0 0" rpy="0 0 0"/>
     <geometry>
-      <mesh filename="file://$(find vector_description)/meshes/base_link.stl" scale="0.001 0.001 0.001"/>
-    </geometry>
-    <material name="white"/>
-  </visual>
-  <!-- No body collision box — only wheels and casters should touch the ground.
-       A body box would scrape the ground during turns and cause wobble. -->
+      <mesh filename="file://$(find vector_description)/meshes/base_bottom.stl" scale="0.001 0.001 0.001"/>
+    </geometry>
+    <material name="grey"/>
+  </visual>
+  <visual name="base_column_visual">
+    <origin xyz="0 0 0" rpy="0 0 0"/>
+    <geometry>
+      <mesh filename="file://$(find vector_description)/meshes/base_column.stl" scale="0.001 0.001 0.001"/>
+    </geometry>
+    <material name="black"/>
+  </visual>
   <collision name="rear_caster_collision">
     <origin xyz="-0.18 0.0 0.0195" rpy="0 0 0"/>
@@ -44,5 +43,5 @@
       <sphere radius="0.02"/>
     </geometry>
-    <material name="dark_grey"/>
+    <material name="black"/>
   </visual>
   <visual name="front_caster_visual">
@@ -51,35 +50,35 @@
       <sphere radius="0.02"/>
     </geometry>
+    <material name="black"/>
+  </visual>
+</link>
+<link name="slider_1">
+  <inertial>
+    <origin xyz="0.0 0.0 0.0" rpy="0 0 0"/>
+    <mass value="0.2"/>
+    <inertia ixx="0.001" iyy="0.001" izz="0.001" ixy="0" iyz="0" ixz="0"/>
+  </inertial>
+  <visual>
+    <origin xyz="-0.131878 -0.005317 -1.244" rpy="0 0 0"/>
+    <geometry>
+      <mesh filename="file://$(find vector_description)/meshes/slider_1.stl" scale="0.001 0.001 0.001"/>
+    </geometry>
+    <material name="black"/>
+  </visual>
+</link>
+<link name="torso_1">
+  <inertial>
+    <origin xyz="0.0 0.0 0.0" rpy="0 0 0"/>
+    <mass value="0.2"/>
+    <inertia ixx="0.001" iyy="0.001" izz="0.001" ixy="0" iyz="0" ixz="0"/>
+  </inertial>
+  <visual>
+    <origin xyz="-0.15 0.0 -0.991427" rpy="0 0 0"/>
+    <geometry>
+      <mesh filename="file://$(find vector_description)/meshes/torso_1.stl" scale="0.001 0.001 0.001"/>
+    </geometry>
     <material name="dark_grey"/>
   </visual>
 </link>
-<link name="slider_1">
-  <inertial>
-    <origin xyz="0.0 0.0 0.0" rpy="0 0 0"/>
-    <mass value="0.2"/>
-    <inertia ixx="0.001" iyy="0.001" izz="0.001" ixy="0" iyz="0" ixz="0"/>
-  </inertial>
-  <visual>
-    <origin xyz="-0.131878 -0.005317 -1.244" rpy="0 0 0"/>
-    <geometry>
-      <mesh filename="file://$(find vector_description)/meshes/slider_1.stl" scale="0.001 0.001 0.001"/>
-    </geometry>
-    <material name="black"/>
-  </visual>
-</link>
-<link name="torso_1">
-  <inertial>
-    <origin xyz="0.0 0.0 0.0" rpy="0 0 0"/>
-    <mass value="0.2"/>
-    <inertia ixx="0.001" iyy="0.001" izz="0.001" ixy="0" iyz="0" ixz="0"/>
-  </inertial>
-  <visual>
-    <origin xyz="-0.15 0.0 -0.991427" rpy="0 0 0"/>
-    <geometry>
-      <mesh filename="file://$(find vector_description)/meshes/torso_1.stl" scale="0.001 0.001 0.001"/>
-    </geometry>
-    <material name="silver"/>
-  </visual>
-</link>
 <link name="left_arm_link_1_1">
   <inertial>
@@ -93,5 +92,5 @@
       <mesh filename="file://$(find vector_description)/meshes/left_arm_link_1_1.stl" scale="0.001 0.001 0.001"/>
     </geometry>
-    <material name="black"/>
+    <material name="silver"/>
   </visual>
 </link>
@@ -107,5 +106,5 @@
       <mesh filename="file://$(find vector_description)/meshes/left_shoulder_1.stl" scale="0.001 0.001 0.001"/>
     </geometry>
-    <material name="black"/>
+    <material name="silver"/>
   </visual>
 </link>
@@ -121,5 +120,5 @@
       <mesh filename="file://$(find vector_description)/meshes/right_arm_link_1_1.stl" scale="0.001 0.001 0.001"/>
     </geometry>
-    <material name="black"/>
+    <material name="silver"/>
   </visual>
 </link>
@@ -135,5 +134,5 @@
       <mesh filename="file://$(find vector_description)/meshes/right_shoulder_1.stl" scale="0.001 0.001 0.001"/>
     </geometry>
-    <material name="black"/>
+    <material name="silver"/>
   </visual>
 </link>
@@ -149,5 +148,5 @@
       <mesh filename="file://$(find vector_description)/meshes/right_bicep_1.stl" scale="0.001 0.001 0.001"/>
     </geometry>
-    <material name="white"/>
+    <material name="silver"/>
   </visual>
 </link>
@@ -163,5 +162,5 @@
       <mesh filename="file://$(find vector_description)/meshes/left_bicep_1.stl" scale="0.001 0.001 0.001"/>
     </geometry>
-    <material name="white"/>
+    <material name="silver"/>
   </visual>
 </link>
@@ -177,5 +176,5 @@
       <mesh filename="file://$(find vector_description)/meshes/right_forearm_v1_1.stl" scale="0.001 0.001 0.001"/>
     </geometry>
-    <material name="white"/>
+    <material name="silver"/>
   </visual>
 </link>
@@ -191,5 +190,5 @@
       <mesh filename="file://$(find vector_description)/meshes/left_forearm_v2_1.stl" scale="0.001 0.001 0.001"/>
     </geometry>
-    <material name="white"/>
+    <material name="silver"/>
   </visual>
 </link>
@@ -205,5 +204,5 @@
       <mesh filename="file://$(find vector_description)/meshes/neck_v2_1.stl" scale="0.001 0.001 0.001"/>
     </geometry>
-    <material name="silver"/>
+    <material name="black"/>
   </visual>
 </link>
@@ -287,5 +286,5 @@
       <mesh filename="file://$(find vector_description)/meshes/left_hand_palm_1.stl" scale="0.001 0.001 0.001"/>
     </geometry>
-    <material name="silver"/>
+    <material name="dark_grey"/>
   </visual>
 </link>
@@ -301,21 +300,21 @@
       <mesh filename="file://$(find vector_description)/meshes/left_hand_finger_1.stl" scale="0.001 0.001 0.001"/>
     </geometry>
+    <material name="silver"/>
+  </visual>
+</link>
+<link name="right_hand_palm_1">
+  <inertial>
+    <origin xyz="0.0 0.0 0.0" rpy="0 0 0"/>
+    <mass value="0.2"/>
+    <inertia ixx="0.001" iyy="0.001" izz="0.001" ixy="0" iyz="0" ixz="0"/>
+  </inertial>
+  <visual>
+    <origin xyz="-0.482 0.177 -0.79" rpy="0 0 0"/>
+    <geometry>
+      <mesh filename="file://$(find vector_description)/meshes/right_hand_palm_1.stl" scale="0.001 0.001 0.001"/>
+    </geometry>
     <material name="dark_grey"/>
   </visual>
 </link>
-<link name="right_hand_palm_1">
-  <inertial>
-    <origin xyz="0.0 0.0 0.0" rpy="0 0 0"/>
-    <mass value="0.2"/>
-    <inertia ixx="0.001" iyy="0.001" izz="0.001" ixy="0" iyz="0" ixz="0"/>
-  </inertial>
-  <visual>
-    <origin xyz="-0.482 0.177 -0.79" rpy="0 0 0"/>
-    <geometry>
-      <mesh filename="file://$(find vector_description)/meshes/right_hand_palm_1.stl" scale="0.001 0.001 0.001"/>
-    </geometry>
-    <material name="silver"/>
-  </visual>
-</link>
 <link name="right_hand_finger_1">
   <inertial>
@@ -329,5 +328,5 @@
       <mesh filename="file://$(find vector_description)/meshes/right_hand_finger_1.stl" scale="0.001 0.001 0.001"/>
     </geometry>
-    <material name="dark_grey"/>
+    <material name="silver"/>
   </visual>
 </link>
@@ -337,7 +336,4 @@
   <child link="slider_1"/>
   <axis xyz="0.0 0.0 1.0"/>
-  <!-- effort raised from 100→2000 to match PID max_effort.
-       Old value of 100 was barely above gravity (78N), leaving no margin.
-       damping=500 prevents instant free-fall during the 5s controller startup. -->
   <limit upper="0.4" lower="-0.6" effort="2000" velocity="100"/>
   <dynamics damping="50.0" friction="10.0"/>

Commit message: added shoulder pads, still misaligned

File: sim/vector_description/urdf/materials.xacro (robot description, xacro)
@@ -6,4 +6,7 @@
 <material name="white">
   <color rgba="1.000 1.000 1.000 1.000"/>
+</material>
+<material name="light_grey">
+  <color rgba="0.900 0.900 0.900 1.000"/>
 </material>
 <material name="dark_grey">

File: sim/vector_description/urdf/vector.xacro (robot description, xacro)
@@ -20,7 +20,7 @@
   </visual>
   <visual name="base_column_visual">
-    <origin xyz="0 0 0" rpy="0 0 0"/>
-    <geometry>
-      <mesh filename="file://$(find vector_description)/meshes/base_column.stl" scale="0.001 0.001 0.001"/>
+    <origin xyz="0 0 -0.0605" rpy="0 0 0"/>
+    <geometry>
+      <mesh filename="file://$(find vector_description)/meshes/base_column.stl" scale="0.001 0.001 0.00125"/>
     </geometry>
     <material name="black"/>
@@ -65,4 +65,32 @@
     </geometry>
     <material name="dark_grey"/>
+  </visual>
+  <visual name="front_left_shoulder_cover">
+    <origin xyz="0.03828 0.191 0.071815" rpy="0 0 0"/>
+    <geometry>
+      <mesh filename="file://$(find vector_description)/meshes/shoulder_cover.stl" scale="0.00025 0.00025 0.00025"/>
+    </geometry>
+    <material name="light_grey"/>
+  </visual>
+  <visual name="back_left_shoulder_cover">
+    <origin xyz="0.03828 0.191 0.071815" rpy="0 0 3.14159265"/>
+    <geometry>
+      <mesh filename="file://$(find vector_description)/meshes/shoulder_cover.stl" scale="0.00025 0.00025 0.00025"/>
+    </geometry>
+    <material name="light_grey"/>
+  </visual>
+  <visual name="front_right_shoulder_cover">
+    <origin xyz="0.03828 -0.186642 0.071815" rpy="0 0 0"/>
+    <geometry>
+      <mesh filename="file://$(find vector_description)/meshes/shoulder_cover.stl" scale="0.00025 0.00025 0.00025"/>
+    </geometry>
+    <material name="light_grey"/>
+  </visual>
+  <visual name="back_right_shoulder_cover">
+    <origin xyz="0.03828 -0.186642 0.071815" rpy="0 0 3.14159265"/>
+    <geometry>
+      <mesh filename="file://$(find vector_description)/meshes/shoulder_cover.stl" scale="0.00025 0.00025 0.00025"/>
+    </geometry>
+    <material name="light_grey"/>
   </visual>
 </link>
