Commit message: added cuboidal base_bottom

File: sim/vector_description/urdf/vector.xacro (robot description, xacro)
@@ -13,7 +13,7 @@
   </inertial>
   <visual name="base_bottom_visual">
-    <origin xyz="0 0 0" rpy="0 0 0"/>
-    <geometry>
-      <mesh filename="file://$(find vector_description)/meshes/base_bottom.stl" scale="0.001 0.001 0.001"/>
+    <origin xyz="-0.212176 -0.203 -0.0275" rpy="0 0 0"/>
+    <geometry>
+      <mesh filename="file://$(find vector_description)/meshes/base_bottomkaran.stl" scale="0.001 0.001 0.001"/>
     </geometry>
     <material name="grey"/>
@@ -38,18 +38,4 @@
     </geometry>
   </collision>
-  <visual name="rear_caster_visual">
-    <origin xyz="-0.18 0.0 0.0175" rpy="0 0 0"/>
-    <geometry>
-      <sphere radius="0.02"/>
-    </geometry>
-    <material name="black"/>
-  </visual>
-  <visual name="front_caster_visual">
-    <origin xyz="0.18 0.0 0.0175" rpy="0 0 0"/>
-    <geometry>
-      <sphere radius="0.02"/>
-    </geometry>
-    <material name="black"/>
-  </visual>
 </link>
 <link name="slider_1">
@@ -428,5 +414,5 @@
   <parent link="base_link"/>
   <child link="right_wheel_1"/>
-  <axis xyz="0.0 -1.0 0.0"/>
+  <axis xyz="0.0 1.0 0.0"/>
 </joint>
 <joint name="left_wheel" type="continuous">

Commit message: added better shoulder cap

File: sim/vector_description/urdf/vector.xacro (robot description, xacro)
@@ -67,28 +67,14 @@
   </visual>
   <visual name="front_left_shoulder_cover">
-    <origin xyz="0.03828 0.191 0.071815" rpy="0 0 0"/>
-    <geometry>
-      <mesh filename="file://$(find vector_description)/meshes/shoulder_cover.stl" scale="0.00025 0.00025 0.00025"/>
+    <origin xyz="0.06143 0.127821 0.071815" rpy="0 0 0"/>
+    <geometry>
+      <mesh filename="file://$(find vector_description)/meshes/shoulder_cover2.stl" scale="0.00025 0.00025 0.00025"/>
     </geometry>
     <material name="light_grey"/>
   </visual>
-  <visual name="back_left_shoulder_cover">
-    <origin xyz="0.03828 0.191 0.071815" rpy="0 0 3.14159265"/>
-    <geometry>
-      <mesh filename="file://$(find vector_description)/meshes/shoulder_cover.stl" scale="0.00025 0.00025 0.00025"/>
-    </geometry>
-    <material name="light_grey"/>
-  </visual>
-  <visual name="front_right_shoulder_cover">
-    <origin xyz="0.03828 -0.186642 0.071815" rpy="0 0 0"/>
-    <geometry>
-      <mesh filename="file://$(find vector_description)/meshes/shoulder_cover.stl" scale="0.00025 0.00025 0.00025"/>
-    </geometry>
-    <material name="light_grey"/>
-  </visual>
   <visual name="back_right_shoulder_cover">
-    <origin xyz="0.03828 -0.186642 0.071815" rpy="0 0 3.14159265"/>
-    <geometry>
-      <mesh filename="file://$(find vector_description)/meshes/shoulder_cover.stl" scale="0.00025 0.00025 0.00025"/>
+    <origin xyz="0.06143 -0.127821 0.071815" rpy="0 0 3.14159265"/>
+    <geometry>
+      <mesh filename="file://$(find vector_description)/meshes/shoulder_cover2.stl" scale="0.00025 0.00025 0.00025"/>
     </geometry>
     <material name="light_grey"/>

Commit message: perfect shoulder commit

File: sim/vector_description/urdf/vector.xacro (robot description, xacro)
@@ -67,14 +67,14 @@
   </visual>
   <visual name="front_left_shoulder_cover">
-    <origin xyz="0.06143 0.127821 0.071815" rpy="0 0 0"/>
-    <geometry>
-      <mesh filename="file://$(find vector_description)/meshes/shoulder_cover2.stl" scale="0.00025 0.00025 0.00025"/>
+    <origin xyz="0.01643 0.240 0.041815" rpy="0 0 0"/>
+    <geometry>
+      <mesh filename="file://$(find vector_description)/meshes/shouldercover3.stl" scale="0.00025 0.00025 0.00025"/>
     </geometry>
     <material name="light_grey"/>
   </visual>
   <visual name="back_right_shoulder_cover">
-    <origin xyz="0.06143 -0.127821 0.071815" rpy="0 0 3.14159265"/>
-    <geometry>
-      <mesh filename="file://$(find vector_description)/meshes/shoulder_cover2.stl" scale="0.00025 0.00025 0.00025"/>
+    <origin xyz="0.10643 -0.240 0.041815" rpy="0 0 3.14159265"/>
+    <geometry>
+      <mesh filename="file://$(find vector_description)/meshes/shouldercover3.stl" scale="0.00025 0.00025 0.00025"/>
     </geometry>
     <material name="light_grey"/>

Commit message: thicker base and added lidar

File: sim/vector_description/urdf/vector.xacro (robot description, xacro)
@@ -22,5 +22,5 @@
     <origin xyz="0 0 -0.0605" rpy="0 0 0"/>
     <geometry>
-      <mesh filename="file://$(find vector_description)/meshes/base_column.stl" scale="0.001 0.001 0.00125"/>
+      <mesh filename="file://$(find vector_description)/meshes/base_column.stl" scale="0.0015 0.0015 0.00125"/>
     </geometry>
     <material name="black"/>
@@ -245,4 +245,37 @@
   </visual>
 </link>
+<!-- INSERT THIS FOR NEW GAZEBO ENGINE OVERRIDES -->
+<gazebo reference="head_v1_1">
+  <visual>
+    <material>
+      <ambient>1 1 1 0</ambient>
+      <diffuse>1 1 1 0</diffuse>
+      <specular>0 0 0 0</specular>
+      <emissive>0 0 0 0</emissive>
+    </material>
+  </visual>
+</gazebo>
+<link name="livox_mid360_link">
+  <inertial>
+    <origin xyz="0.0 0.0 0.0" rpy="0 0 0"/>
+    <mass value="0.265"/>
+    <inertia ixx="0.0002" iyy="0.0002" izz="0.0003" ixy="0" iyz="0" ixz="0"/>
+  </inertial>
+  <visual name="livox_mid360_visual">
+    <origin xyz="0 0 0" rpy="0 0 0"/>
+    <geometry>
+      <cylinder radius="0.053" length="0.052"/>
+    </geometry>
+    <material name="dark_grey"/>
+  </visual>
+</link>
+<joint name="livox_mid360_joint" type="fixed">
+  <!-- Mounted on top of the base column, just below the slider mechanism.
+       slider_1 origin is at (0.131878, 0.005317, 1.244) from base_link,
+       so we offset back to center the LiDAR on the column axis. -->
+  <origin xyz="-0.131878 -0.005317 -0.01" rpy="0 0 0"/>
+  <parent link="slider_1"/>
+  <child link="livox_mid360_link"/>
+</joint>
 <link name="right_wheel_1">
   <inertial>

Commit message: removed head and fixed the pointcloud2 flickering

File: sim/vector_description/urdf/vector.xacro (robot description, xacro)
@@ -294,5 +294,5 @@
     <origin xyz="0 0 0" rpy="1.5707963 0 0"/>
     <geometry>
-      <sphere radius="0.075"/>
+      <cylinder radius="0.075" length="0.08"/>
     </geometry>
   </collision>
@@ -314,5 +314,5 @@
     <origin xyz="0 0 0" rpy="1.5707963 0 0"/>
     <geometry>
-      <sphere radius="0.075"/>
+      <cylinder radius="0.075" length="0.08"/>
     </geometry>
   </collision>
